File: ОИиЦЭ/лаба Н/лаба.kicad_sch (KiCad schematic)
At the start: 40 parts

Commit message: Муфта конец
Parts:
- removed DD1.2, DD1.3: ~, symbol LOG:Инвертор
- removed DD2.2: ~, symbol LOG:3входа
- removed DD3.1: ~, symbol LOG:2входа
- added DD2.1, DD2.2, DD2.3: ~, symbol LOG:Инвертор_2_входа
- renumbered DD2.1 to DD1.1
Connections:
- net at DD1.2.: now also DD1.3.; no longer DD2.2.
- net at DD1.3.: now also DD2.1.; no longer DD1.2.
- net at DD1.1.: now also DD2.2. (x3)
- net at DD2.3.: now also DD1.4.
- net at DD1.4.: now also DD1.3.; no longer DD2.3.
- net at DD2.2.: now also DD2.1.; no longer DD1.1.
- net at DD1.3.: now also DD1.2., R3.2
- net at DD2.1.: now also DD2.3.; no longer DD1.1.
- net at DD2.4.: now also DD2.3.; no longer DD1.1.
- net at DD2.2.: now also DD2.3.; no longer DD1.1.
- net at DD2.3.: now also R2.2
- new net: DD1.2., DD2.2.
- new net: DD3.2., DD3.4., DD3.5., R1.2
- new net: DD1.1., DD2.1. (x3)
- new net: DD1.4., DD2.2.
- new net: DD1.1., DD2.4.
- new net: DD2.1., DD2.2.
- new net: DD2.2., DD2.3.
- now unconnected: DD1.2., DD3.2., DD3.4., DD3.5.
Other:
- note added: "3 1 2"
- note added: "6 4 5"
- note added: "Схема на различных ЛЭ DD1 - К555ЛИ3 DD2 - К555ЛЕ1"
- note removed: "1 2"
- note removed: "3 4"
- note removed: "Схема на различных ЛЭ DD1 - К555ЛН1 DD2 - К555ЛИ3 DD3 - К555ЛЛ1"
- moved on the sheet: DD1.1
