File: KiCad/КР1156ЕУ5 Повыш/КР1156ЕУ5 Повыш.kicad_sch (KiCad schematic)
At the start: 10 parts, among them U1 КР1156ЕУ5

Commit message: KF
Parts:
- removed C1: 100u, symbol Device:C
- removed C2: 1500, symbol Device:C
- removed C3: 330u, symbol Device:C
- removed L1: 175u, symbol Device:L
- removed R1: 0.22, symbol Device:R
- removed R2: 47k, symbol Device:R
- removed R3: 2.2, symbol Device:R
- removed R4: 180, symbol Device:R
- removed U1: КР1156ЕУ5, Package_SO:SOIC-8_3.9x4.9mm_P1.27mm, symbol work:MC33063AD
- added DА1: ~, symbol for work:КР1156ЕУ5
- added Input: ~, symbol for work:terminal_block_input
- added L2: 170u, symbol for work:Inductor
- added R4: 180, symbol for work:Resistor
- added R6, R7: ~, symbol for work:Resistor
- added С1: 100u, symbol for work:Capacitor
- added С2: 1500n, symbol for work:Capacitor
- added С3: 330u, symbol for work:Capacitor
- renumbered D1 to VD1
Connections:
- net at VD1.1 (K): now also R6., С3.
- net at VD1.2 (A): now also DА1.1 (C_OUT ), L2.
- new net: DА1.2 (E_OUT), DА1.4 (GND), С2.
- new net: DА1.3 (TC), С2.
- new net: DА1.5 (CMP), R6., R7.
- new net: DА1.6 (Vcc), DА1.7 (Rt), L2., R4., С1.
- new net: DА1.8 (DRC), R4.
Other:
- moved on the sheet: VD1

Commit message: писька-отвалиська
Parts:
- removed Input: ~, symbol for work:terminal_block_input
- removed L2: 170u, symbol for work:Inductor
- removed R4: 180, symbol for work:Resistor
- removed R6, R7: ~, symbol for work:Resistor
- removed VD1: 1N5819, Diode_THT:D_DO-41_SOD81_P10.16mm_Horizontal, symbol Diode:1N5819
- removed С1: 100u, symbol for work:Capacitor
- removed С2: 1500n, symbol for work:Capacitor
- removed С3: 330u, symbol for work:Capacitor
- added C1: smd-конденсатор-тантал*68мк*10В*D*ВП, KICAD6_RLC:Конденсатор_тантал_SMD_m7343, symbol niisk_lib_C:smd-конденсатор-тантал*68мк*10В*D*ВП
- added C2: smd-конденсатор-керамика*1,5мк*25В*1812*ВП, KICAD6_RLC:Конденсатор_SMD_IEC_1812, symbol niisk_lib_C:smd-конденсатор-керамика*1,5мк*25В*1812*ВП
- added C3: dip-конденсатор-электролит*470мк*35В*D10x17-гориз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, KICAD6_RLC:Конденсатор_электролит_DIP_d10х17_horizontal, symbol IMPORT:dip-конденсатор-электролит*470мк*35В*D10x17-горизонтальный*импорт
- added L1: smd-индуктивность*47мкГн*0,24А*1812*ВП, MOTOR_RLC:Индуктивность_МД43Ф(1812), symbol niisk_lib:smd-индуктивность*47мкГн*0,24А*1812*ВП
- added R1: smd-резистор*0,01*2512*ВП, MOTOR_RLC:Резистор_SMD_2512-1,0_Вт, symbol niisk_lib:smd-резистор*0,01*2512*ВП
- added R2: smd-резистор*47*2Вт*5проц*4020*ВП, KICAD6_RLC:Резистор_SMD_IEC_4020-2,0_Вт, symbol niisk_lib_R:smd-резистор*47*2Вт*5проц*4020*ВП
- added R3: smd-резистор*2,2*1Вт*5проц*2512*ВП, KICAD6_RLC:Резистор_SMD_IEC_2512-1,0_Вт, symbol niisk_lib_R:smd-резистор*2,2*1Вт*5проц*2512*ВП
- added R4: smd-резистор*180к*0,1Вт*5проц*0603*ВП, KICAD6_RLC:Резистор_SMD_IEC_0603-0,1_Вт, symbol niisk_lib_R:smd-резистор*180к*0,1Вт*5проц*0603*ВП
- added VD2: Ограничитель_напряжения*2Р244А91*6,4В*10мА*ОТК, MOTOR_VD_VT_HL:Диод_SMB, symbol niisk_lib_V:Ограничитель_напряжения*2Р244А91*6,4В*10мА*ОТК
- added XT1, XT2, XT3, XT4: dip-клемма*серая*1контакт*16А*шаг5мм*олово*ВП, MOTOR_X:СКПП-2,5-1-2-05, symbol niisk_lib:dip-клемма*серая*1контакт*16А*шаг5мм*олово*ВП
- DА1: footprint (none) -> MOTOR_DD:DIP8
Connections:
- net at DА1.1 (C_OUT ): now also L1.2, VD2.1 (АНОД)
- net GND: now reaches DА1.2 (E_OUT), DА1.4 (GND)
- net GND: now also C1.1, C2.2, C3.2, R3.1, XT2.1, XT4.1
- net at DА1.3 (EXT_CAP): now also C2.1
- net at DА1.5 (FB): now also R2.1, R3.2
- net at DА1.6 (VCC(3-40B)): now also C1.2, R1.1, XT1.1; no longer DА1.7 (Rt)
- net at DА1.8 (C_IN): now also R4.2
- new net: DА1.7 (CUR_SENS), L1.1, R1.2, R4.1
- new net: C3.1, R2.2, VD2.2 (КАТОД), XT3.1
