File: KiCad/КР1156ЕУ5 Повыш/КР1156ЕУ5 Повыш.kicad_pcb (KiCad board)
At the start: 2 copper layers, 13 parts

Commit message: Повышайка конепц, Курсач усе
Parts:
- removed DА1: ~, MOTOR_DD:DIP8
- removed VD2: Ограничитель_напряжения*2Р244А91*6,4В*10мА*ОТК, MOTOR_VD_VT_HL:Диод_SMB
- removed XT1, XT2, XT3, XT4: dip-клемма*серая*1контакт*16А*шаг5мм*олово*ВП, MOTOR_X:СКПП-2,5-1-2-05
- added G1: ~, for_work:DIP8, F.Cu at (153.5, 114.2)
- added R1: ~, for_work:1206, F.Cu at (138.2, 118.2)
- added VD1: ~, for_work:VD, F.Cu at (167.0, 118.2)
- added XP1: ~, for_work:Клеммник наборный, F.Cu at (131.0, 112.0)
- added XP2: ~, for_work:Клеммник наборный, F.Cu at (181.5, 117.0)
- C1: value smd-конденсатор-тантал*68мк*10В*D*ВП -> 1.5мк; footprint KICAD6_RLC:Конденсатор_тантал_SMD_m7343 -> for_work:0805
- C2: value smd-конденсатор-керамика*1,5мк*25В*1812*ВП -> 1.5мк; footprint KICAD6_RLC:Конденсатор_SMD_IEC_1812 -> for_work:0805
- C3: value dip-конденсатор-электролит*470мк*35В*D10x17-горизонтальный*импорт -> 1.5мк; footprint KICAD6_RLC:Конденсатор_электролит_DIP_d10х17_horizontal -> for_work:С_0810
- L1: value smd-индуктивность*47мкГн*0,24А*1812*ВП -> Чип_индуктивность*10000н*50В*ВП; footprint MOTOR_RLC:Индуктивность_МД43Ф(1812) -> MOTOR_RLC:Чип-индуктивность_SMD_0805
- R2: value smd-резистор*47*2Вт*5проц*4020*ВП -> ~; footprint KICAD6_RLC:Резистор_SMD_IEC_4020-2,0_Вт -> for_work:0805
- R3: value smd-резистор*2,2*1Вт*5проц*2512*ВП -> ~; footprint KICAD6_RLC:Резистор_SMD_IEC_2512-1,0_Вт -> for_work:0805
- R4: value smd-резистор*180к*0,1Вт*5проц*0603*ВП -> ~; footprint KICAD6_RLC:Резистор_SMD_IEC_0603-0,1_Вт -> for_work:0805
- moved R2 54.7 mm to (159.0, 107.5)
- moved C1 48.3 mm to (136.8, 112.2), turned to 90 degrees
- moved C3 47.5 mm to (172.2, 102.8)
- moved R3 46.4 mm to (145.5, 107.5), turned to 0 degrees
- moved R4 45.3 mm to (145.0, 118.2)
- moved C2 43.9 mm to (161.2, 113.2)
- moved L1 43.0 mm to (152.5, 123.0)
Connections:
- C1 pad 1: GND -> Net-(G1-VCC(3-40В))
- C1 pad 2: Net-(DА1-VCC(3-40B)) -> GND
- C3 pad 1: Net-(VD2-КАТОД) -> GND
- C3 pad 2: GND -> Net-(C3-Pad2)
- R2 pad 2: Net-(VD2-КАТОД) -> Net-(C3-Pad2)
Routing:
- net GND: track 200.1 -> 26.6 mm, vias 0 -> 2
- net Net-(VD2-КАТОД): track 55.4 -> 0.00 mm
- net Net-(C3-Pad2): track 0.00 -> 41.2 mm
- net Net-(G1-VCC(3-40В)): track 0.00 -> 23.8 mm
- net Net-(DА1-VCC(3-40B)): track 23.0 -> 0.00 mm
- net Net-(G1-FB): track 24.7 -> 17.4 mm
- net Net-(G1-C_OUT): track 17.9 -> 14.8 mm
- net Net-(G1-EXT_CAP): track 5.44 -> 3.00 mm
- net Net-(G1-CUR_SENS): track 32.0 -> 30.0 mm
- net Net-(G1-C_IN): track 4.45 -> 3.75 mm
- added copper zone on B.Cu, net GND
