File: sem8/БЦВКУРКА/БЦВКУ РКА Э3/БЦВКУ РКА Э3.kicad_sch (KiCad schematic)
At the start: 26 parts

Commit message: Деркач БЦВКУ
Parts:
- added K1, K2: ~, symbol dwgn:Реле
- added R7, R9: smd-резистор*1,5к*1Вт*5проц*2512*ВП, MTR_KICAD_RLC:Резистор_SMD_2512_IEC_61188-5-2(ур.2), symbol mtr_kicad_R:smd-резистор*1,5к*1Вт*5проц*2512*ВП
- added VT5, VT6: Транзистор NPN КТ229Г9, KICAD7_V:SOT-23-3-LikeTSOP2-300mil_IEC_61188-5-3(ур.2), symbol kicad7_V:smd-транзистор*npn*0,5А*45В*КТ-46(SOT-23)*ОТК
- added XT6, XT9: Соединитель клеммный пружинный СКПП-1,0-5Г-2х1-3-К, KICAD7_X:Клеммник_DG390-5.0_DaSh, symbol kicad7_X:dip-клемма-нажимная*СКПП-1,0*2контакта*10А*шаг5мм*олово*ОТК
Connections:
- net 0V: now also HL1.K, VT5.2, VT6.2, XT6.2, XT9.2; no longer HL1.A, SA1.2
- net LED0: now also HL2.K; no longer HL2.A
- net LED1: now also HL3.K; no longer HL3.A
- net RST: no longer R3., VD1.K
- net at R5.: no longer HL2.K
- net at R6.: now also HL3.A
- net at R4.: no longer HL1.K
- net at R8.: now also XT5.2
- new net: HL2.A, R5.
- new net: R3., SA1.2
- new net: R9., VT5.1
- new net: K2., XT6.1
- new net: K2., VT6.3
- new net: R7., VT6.1
- new net: K1., VT5.3
- new net: K1., XT9.1
- new net: HL1.A, R4.
- no-connect marks 0 -> 2
Other:
- moved on the sheet: C1, C2, HL1, HL2, HL3, R3, R4, SA1, VT3, VT4, XT2, ZQ1
